Commit message: regular update

File: src/common/urdf/base.urdf (robot description, URDF)
Before this commit: robot base, 3 links, 2 joints
Links:
- added link imu; visual cylinder length=0.01 radius=0.01
Joints:
- added joint base_to_imu: type fixed, parent base_link, child imu, origin xyz=0 0 0.3

Commit message: update

File: src/common/urdf/base.urdf (robot description, URDF)
Before this commit: robot base, 4 links, 3 joints
Links:
- removed link point
- link base_link: geometry visual cylinder length=0.2 radius=0.26
- link laser: geometry visual cylinder length=0.08 radius=0.08
Joints:
- removed joint base_to_point
- joint base_to_imu: origin xyz=0 0 0.3 -> xyz=0 0 0.2
- joint base_to_laser: origin xyz=0.3 0 0.2 -> xyz=0.2 0 0.2
